Commit message: stash

File: ros2_ws/src/robot_description/urdf/arm_only_franka.urdf (robot description, URDF)
Before this commit: robot mobile_base_with_franka, 19 links, 18 joints
Links:
- removed link bumblebee_stereo_left_camera
- removed link bumblebee_stereo_right_camera
- removed link front_left_wheel_link
- removed link front_right_wheel_link
- removed link imu_sensor
- removed link odom
- removed link rear_left_wheel_link
- removed link rear_right_wheel_link
- added link arm_base; collision box size=0.42 0.31 0.184
Joints:
- removed joint car_to_franka_fixed
- removed joint front_left_wheel_joint
- removed joint front_right_wheel_joint
- removed joint joint_odom-bumblebee_stereo_left_camera
- removed joint joint_odom-bumblebee_stereo_right_camera
- removed joint joint_odom-imu_sensor
- removed joint rear_left_wheel_joint
- removed joint rear_right_wheel_joint
- added joint arm_base_to_panda_fixed: type fixed, parent arm_base, child panda_panda_link0, origin xyz=-0.055 0 0.19 rpy=0 0 0

Commit message: 使用setup assistant配置完成，demo.launch.py work well

File: ros2_ws/src/robot_description/urdf/arm_only_franka.urdf (robot description, URDF)
Before this commit: robot arm_only_franka, 12 links, 11 joints
Links:
- removed link panda_panda_hand
- removed link panda_panda_leftfinger
- removed link panda_panda_link0
- removed link panda_panda_link1
- removed link panda_panda_link2
- removed link panda_panda_link3
- removed link panda_panda_link4
- removed link panda_panda_link5
- removed link panda_panda_link6
- removed link panda_panda_link7
- removed link panda_panda_rightfinger
- added link panda_hand, mass 0.5583305; collision mesh filename=file:///data/project/isaac_test/meshesfranka/panda_hand_geo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 scale=1. 1. 1.; visual mesh filename=file:///data/project/isaac_test/meshesfranka/panda_hand_geo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 scale=1. 1. 1.
- added link panda_leftfinger, mass 0.0140552; collision mesh filename=file:///data/project/isaac_test/meshesfranka/panda_leftfing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 scale=1. 1. 1.; visual mesh filename=file:///data/project/isaac_test/meshesfranka/panda_leftfing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 scale=1. 1. 1.
- added link panda_link0, mass 2.8142028; collision mesh filename=file:///data/project/isaac_test/meshesfranka/panda_link0_ge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 scale=1. 1. 1.; visual mesh filename=file:///data/project/isaac_test/meshesfranka/panda_link0_ge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 scale=1. 1. 1.
- added link panda_link1, mass 2.3599997; collision mesh filename=file:///data/project/isaac_test/meshesfranka/panda_link1_ge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 scale=1. 1. 1.; visual mesh filename=file:///data/project/isaac_test/meshesfranka/panda_link1_ge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 scale=1. 1. 1.
- added link panda_link2, mass 2.3795187; collision mesh filename=file:///data/project/isaac_test/meshesfranka/panda_link2_ge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 scale=1. 1. 1.; visual mesh filename=file:///data/project/isaac_test/meshesfranka/panda_link2_ge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 scale=1. 1. 1.
- added link panda_link3, mass 2.6498823; collision mesh filename=file:///data/project/isaac_test/meshesfranka/panda_link3_ge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 scale=1. 1. 1.; visual mesh filename=file:///data/project/isaac_test/meshesfranka/panda_link3_ge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 scale=1. 1. 1.
- added link panda_link4, mass 2.6948018; collision mesh filename=file:///data/project/isaac_test/meshesfranka/panda_link4_ge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 scale=1. 1. 1.; visual mesh filename=file:///data/project/isaac_test/meshesfranka/panda_link4_ge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 scale=1. 1. 1.
- added link panda_link5, mass 2.9812818; collision mesh filename=file:///data/project/isaac_test/meshesfranka/panda_link5_ge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 scale=1. 1. 1.; visual mesh filename=file:///data/project/isaac_test/meshesfranka/panda_link5_ge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 scale=1. 1. 1.
- added link panda_link6, mass 1.1285807; collision mesh filename=file:///data/project/isaac_test/meshesfranka/panda_link6_ge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 scale=1. 1. 1.; visual mesh filename=file:///data/project/isaac_test/meshesfranka/panda_link6_ge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 scale=1. 1. 1.
- added link panda_link7, mass 0.4052913; collision mesh filename=file:///data/project/isaac_test/meshesfranka/panda_link7_ge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 scale=1. 1. 1.; visual mesh filename=file:///data/project/isaac_test/meshesfranka/panda_link7_ge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 scale=1. 1. 1.
- added link panda_rightfinger, mass 0.0140552; collision mesh filename=file:///data/project/isaac_test/meshesfranka/panda_rightfin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 scale=1. 1. 1.; visual mesh filename=file:///data/project/isaac_test/meshesfranka/panda_rightfin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 scale=1. 1. 1.
Joints:
- joint arm_base_to_panda_fixed: child panda_panda_link0 -> panda_link0
- joint panda_finger_joint1: child panda_panda_leftfinger -> panda_leftfinger; parent panda_panda_hand -> panda_hand
- joint panda_finger_joint2: child panda_panda_rightfinger -> panda_rightfinger; parent panda_panda_hand -> panda_hand
- joint panda_hand_joint: child panda_panda_hand -> panda_hand; parent panda_panda_link7 -> panda_link7
- joint panda_joint1: child panda_panda_link1 -> panda_link1; parent panda_panda_link0 -> panda_link0
- joint panda_joint2: child panda_panda_link2 -> panda_link2; parent panda_panda_link1 -> panda_link1
- joint panda_joint3: child panda_panda_link3 -> panda_link3; parent panda_panda_link2 -> panda_link2
- joint panda_joint4: child panda_panda_link4 -> panda_link4; parent panda_panda_link3 -> panda_link3
- joint panda_joint5: child panda_panda_link5 -> panda_link5; parent panda_panda_link4 -> panda_link4
- joint panda_joint6: child panda_panda_link6 -> panda_link6; parent panda_panda_link5 -> panda_link5
- joint panda_joint7: child panda_panda_link7 -> panda_link7; parent panda_panda_link6 -> panda_link6

File: ros2_ws/src/robot_description/urdf/combined_car_franka.urdf (robot description, URDF)
Before this commit: robot mobile_base_with_franka, 19 links, 18 joints
Links:
- link odom: mass 17. -> None
