Commit message: 对的

File: ros2_ws/src/robot_description/urdf/combined_car_franka_change.urdf (robot description, URDF)
Before this commit: robot mobile_base_with_franka, 19 links, 18 joints
Joints:
- joint panda_finger_joint1: origin xyz=-0.0584 -0.0000001 -0.  rpy=-1.5707964 -0.7853983 1.5707964 -> xyz=-0.0584 -0.0000001 -0.  rpy=0. 0. 0.7853983
- joint panda_finger_joint2: mimic (none) -> joint=panda_finger_joint1; origin xyz=-0.0584 -0.0000001 -0.  rpy=1.5707964 0.7853983 -1.5707964 -> xyz=-0.0584 -0.0000001 -0.  rpy=0. 0. 0.7853983
- joint panda_joint4: limit lower=-3.0718 upper=-0.0698 effort=87. velocity=2.1749999 -> lower=-3.0718 upper=2.0 effort=87. velocity=2.1749999; origin xyz=-0. -0.0000001 -0.0824999 rpy=-0.0000002 0.0000002 -1.5707968 -> xyz=-0. -0.0000001 -0.0824999 rpy=-0.0000002 0.0000002 0.
