Commit message: simplify the python script and add props, action graph in usd. test well. with correct collision.

File: ros2_ws/src/robot_description/urdf/combined_car_franka.urdf (robot description, URDF)
Before this commit: robot mobile_base_with_franka, 19 links, 18 joints
Joints:
- joint panda_finger_joint2: limit lower=0. upper=0.04 effort=0. velocity=10. -> lower=0. upper=0.04 effort=7.1999998 velocity=0.2
