Commit message: forget to add change

File: ros2_ws/src/moveit_robot_config/config/mobile_base_with_franka.ros2_control.xacro (robot description, xacro)
@@ -1,10 +1,16 @@
 <?xml version="1.0"?>
 <robot xmlns:xacro="http://www.ros.org/wiki/xacro">
-    <xacro:macro name="mobile_base_with_franka_ros2_control" params="name initial_positions_file">
+    <xacro:macro name="mobile_base_with_franka_ros2_control" params="name initial_positions_file ros2_control_hardware_type:='mock_components'">
         <xacro:property name="initial_positions" value="${load_yaml(initial_positions_file)['initial_positions']}"/>
         <ros2_control name="${name}" type="system">
             <hardware>
-                <!-- By default, set up controllers for simulation. This won't work on real hardware -->
-                <plugin>mock_components/GenericSystem</plugin>
+                <xacro:if value="${ros2_control_hardware_type == 'isaac'}">
+                    <plugin>topic_based_ros2_control/TopicBasedSystem</plugin>
+                    <param name="joint_commands_topic">/joint_commands</param>
+                    <param name="joint_states_topic">/joint_states</param>
+                </xacro:if>
+                <xacro:if value="${ros2_control_hardware_type == 'mock_components'}">
+                    <plugin>mock_components/GenericSystem</plugin>
+                </xacro:if>
             </hardware>
             <joint name="panda_joint1">
@@ -65,9 +71,13 @@
             </joint>
             <joint name="panda_finger_joint2">
-                <command_interface name="position"/>
+                <param name="mimic">panda_finger_joint1</param>
+                <param name="multiplier">1</param>
+                <command_interface name="position" />
                 <state_interface name="position">
-                  <param name="initial_value">${initial_positions['panda_finger_joint2']}</param>
+                  <param name="initial_value">0.0</param>
                 </state_interface>
-                <state_interface name="velocity"/>
+                <state_interface name="velocity">
+                    <param name="initial_value">0.0</param>
+                </state_interface>
             </joint>
         </ros2_control>

File: ros2_ws/src/moveit_robot_config/config/mobile_base_with_franka.urdf.xacro (robot description, xacro)
@@ -2,8 +2,9 @@
 <robot xmlns:xacro="http://www.ros.org/wiki/xacro" name="mobile_base_with_franka">
     <xacro:arg name="initial_positions_file" default="initial_positions.yaml" />
+    <xacro:arg name="ros2_control_hardware_type" default="mock_components" />
     <!-- Import mobile_base_with_franka urdf file -->
     <xacro:include filename="$(find robot_description)/urdf/combined_car_franka.urdf" />
     <!-- Import control_xacro -->
     <xacro:include filename="mobile_base_with_franka.ros2_control.xacro" />
-    <xacro:mobile_base_with_franka_ros2_control name="FakeSystem" initial_positions_file="$(arg initial_positions_file)"/>
+    <xacro:mobile_base_with_franka_ros2_control name="FakeSystem" initial_positions_file="$(arg initial_positions_file)" ros2_control_hardware_type="$(arg ros2_control_hardware_type)"/>
 </robot>

Commit message: change the finger2 into mimic joint

File: ros2_ws/src/moveit_robot_config/config/mobile_base_with_franka.ros2_control.xacro (robot description, xacro)
@@ -68,5 +68,7 @@
                   <param name="initial_value">${initial_positions['panda_finger_joint1']}</param>
                 </state_interface>
-                <state_interface name="velocity"/>
+                <state_interface name="velocity">
+                    <param name="initial_value">0.0</param>
+                </state_interface>
             </joint>
             <joint name="panda_finger_joint2">

File: ros2_ws/src/robot_description/urdf/combined_car_franka copy.urdf (robot description, URDF)
Before this commit: robot mobile_base_with_franka, 19 links, 18 joints
Joints:
- joint panda_finger_joint2: mimic joint=panda_finger_joint1 -> (none)
